File: io-gateway/relays.kicad_sch (KiCad schematic)
At the start: 24 parts, among them K1 2071556-2, K2 2071556-2, K3 2071556-2, K4 2071556-2, K5 2071556-2, K6 2071556-2, Q1 NTR4003NT1G, Q2 NTR4003NT1G, Q3 NTR4003NT1G, Q4 NTR4003NT1G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

Commit message: update mcu lib
Parts:
- K1, K2: footprint 20715562 -> Relay:20715562
Changed lines of the file:
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@@
 			)
 		)
-		(property "Footprint" "20715562"
+		(property "Footprint" "Relay:20715562"
 			(at 151.13 152.07 0)
 			(effects
@@
 			)
 		)
-		(property "Footprint" "20715562"
+		(property "Footprint" "Relay:20715562"
 			(at 83.82 150.8 0)
 			(effects
