File: io-gateway/io-gateway.kicad_pcb (KiCad board)
At the start: 4 copper layers, 155 x 81.5 mm, 127 parts, among them IC1 MAX17673AATI+, J1 1752201, J2 1752201, J3 1752201, J4 Screw_Terminal_01x09, J5 Screw_Terminal_01x09, J6 Screw_Terminal_01x09, K1 2071556-2, K10 2071556-2, K11 2071556-2, K12 2071556-2, K13 2071556-2, K14 2071556-2, K15 2071556-2, K16 2071556-2, K17 2071556-2, K18 2071556-2, K2 2071556-2, K3 2071556-2, K4 2071556-2, K5 2071556-2, K6 2071556-2, K7 2071556-2, K8 2071556-2, K9 2071556-2, Q1 NTR4003NT1G, Q10 NTR4003NT1G, Q11 NTR4003NT1G, Q12 NTR4003NT1G, Q13 NTR4003NT1G, Q14 NTR4003NT1G, Q15 NTR4003NT1G, Q16 NTR4003NT1G, Q17 NTR4003NT1G, Q18 NTR4003NT1G, Q2 NTR4003NT1G, Q3 NTR4003NT1G, Q4 NTR4003NT1G, Q5 NTR4003NT1G, Q6 NTR4003NT1G, Q7 NTR4003NT1G, Q8 NTR4003NT1G, Q9 NTR4003NT1G

Commit message: update
Parts:
- removed D11, D12, D13, D14, D15, D16, D17, D18, D19, D9: MMSD914, Diode_SMD:D_SOD-123
- removed K10, K11, K12, K13, K14, K15, K16, K17, K18, K8: 2071556-2, Relays:20715562
- removed Q10, Q11, Q12, Q13, Q14, Q15, Q16, Q17, Q18, Q8: NTR4003NT1G, Package_TO_SOT_SMD:SOT-23-3
- removed R27, R29, R30, R31, R32, R33, R34, R35, R36, R37: 100, Resistor_SMD:R_0603_1608Metric
- added C22: 100nF 50V, Capacitor_SMD:C_0201_0603Metric, F.Cu at (59.9, 166.2)
- added C23: 1µF 50V, Capacitor_SMD:C_1206_3216Metric, F.Cu at (85.9, 138.6)
- added C24: NM, Capacitor_SMD:C_1206_3216Metric, F.Cu at (85.9, 141.9)
- added C25: 22pF, Capacitor_SMD:C_0603_1608Metric, F.Cu at (75.4, 138.1)
- added C26: 470pF, Capacitor_SMD:C_0603_1608Metric, F.Cu at (75.4, 140.6)
- added C27: 10µF 50V, Capacitor_SMD:C_1210_3225Metric, F.Cu at (80.3, 139.0)
- added C28: 10µF 50V, Capacitor_SMD:C_1210_3225Metric, F.Cu at (80.3, 143.2)
- added C29: 100nF 50V, Capacitor_SMD:C_0201_0603Metric, F.Cu at (59.9, 168.0)
- added C30: 10µF 50V, Capacitor_SMD:C_1210_3225Metric, F.Cu at (80.3, 147.5)
- added C31: 10µF 50V, Capacitor_SMD:C_1210_3225Metric, F.Cu at (80.3, 151.8)
- added C32: 470pF, Capacitor_SMD:C_0603_1608Metric, F.Cu at (75.4, 143.2)
- added C33: 100nF 50V, Capacitor_SMD:C_0201_0603Metric, F.Cu at (59.9, 169.8)
- added C34: 22pF, Capacitor_SMD:C_0603_1608Metric, F.Cu at (75.4, 145.7)
- added C35: 100nF 50V, Capacitor_SMD:C_0201_0603Metric, F.Cu at (59.9, 171.5)
- added C36: 1µF 50V, Capacitor_SMD:C_1206_3216Metric, F.Cu at (85.9, 145.2)
- added C37: NM, Capacitor_SMD:C_1206_3216Metric, F.Cu at (85.9, 148.6)
- added D20: D_Zener, Diode_SMD:D_SOD-123, F.Cu at (64.0, 167.1)
- added D21: D_Schottky, Diode_SMD:D_SMB, F.Cu at (86.1, 159.7)
- added D22: D_Schottky, Diode_SMD:D_SMB, F.Cu at (86.1, 165.3)
- added D23: D_Zener, Diode_SMD:D_SOD-123, F.Cu at (64.0, 170.4)
- added L4: 47µH 3.8A, Inductor_SMD:L_12x12mm_H8mm, F.Cu at (79.8, 98.5)
- added L5: 47µH 3.8A, Inductor_SMD:L_12x12mm_H8mm, F.Cu at (93.2, 98.5)
- added R38: 47k, Resistor_SMD:R_0603_1608Metric, F.Cu at (75.4, 148.2)
- added R39: 24k9, Resistor_SMD:R_0603_1608Metric, F.Cu at (75.4, 150.7)
- added R40: 24k9, Resistor_SMD:R_0603_1608Metric, F.Cu at (75.4, 153.2)
- added R41: 47k, Resistor_SMD:R_0603_1608Metric, F.Cu at (75.4, 155.7)
- added RS_DIM1: R, Resistor_SMD:R_1206_3216Metric, F.Cu at (69.7, 167.0)
- added RS_DIM2: R, Resistor_SMD:R_1206_3216Metric, F.Cu at (69.7, 170.3)
- added U1: LED5000, Package_SO:HSOP-8-1EP_3.9x4.9mm_P1.27mm_EP2.41x3.1mm, F.Cu at (77.7, 160.3)
- added U2: LED5000, Package_SO:HSOP-8-1EP_3.9x4.9mm_P1.27mm_EP2.41x3.1mm, F.Cu at (77.7, 166.9)
- moved D4 137.1 mm to (-32.9, 165.1)
- moved D6 137.1 mm to (-45.1, 165.1)
- moved K1 137.1 mm to (-16.6, 165.1)
- moved Q2 137.1 mm to (-37.4, 169.7)
- moved R13 137.1 mm to (-33.2, 168.7)
- moved D10 137.1 mm to (-0.25, 173.4)
- moved D2 137.1 mm to (-20.5, 165.1)
- moved D3 137.1 mm to (-41.0, 173.4)
- moved D5 137.1 mm to (-61.3, 173.4)
- moved D7 137.1 mm to (-57.5, 165.1)
- moved D8 137.1 mm to (20.1, 173.5)
- moved K2 137.1 mm to (-41.0, 177.3)
- moved K3 137.1 mm to (-28.9, 165.1)
- moved K4 137.1 mm to (-61.3, 177.3)
- moved K5 137.1 mm to (-41.2, 165.1)
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Connections:
- net /Terminal Blocks/DIMMER_OUT_2.1 renamed DIM3_VLED+
- net /Terminal Blocks/DIMMER_OUT_2.2 renamed DIM3_VLED-
- net /Terminal Blocks/DIMMER_OUT_2.3 renamed DIM4_VLED+
- net /Terminal Blocks/DIMMER_OUT_2.4 renamed DIM4_VLED-
- net /Terminal Blocks/DIMMER_OUT_3.1 renamed DIM5_VLED+
- net /Terminal Blocks/DIMMER_OUT_3.2 renamed DIM5_VLED-
- net /Terminal Blocks/DIMMER_OUT_3.3 renamed DIM6_VLED+
- net /Terminal Blocks/DIMMER_OUT_3.4 renamed DIM6_VLED-
- net /Terminal Blocks/DIMMER_OUT_4.1 renamed DIM7_VLED+
- net /Terminal Blocks/DIMMER_OUT_4.2 renamed DIM7_VLED-
- net /Terminal Blocks/DIMMER_OUT_4.3 renamed DIM8_VLED+
- net /Terminal Blocks/DIMMER_OUT_4.4 renamed DIM8_VLED-
- net /Terminal Blocks/DIMMER_OUT_5.1 renamed DIM9_VLED+
- net /Terminal Blocks/DIMMER_OUT_5.2 renamed DIM9_VLED-
- net /Terminal Blocks/DIMMER_OUT_5.3 renamed DIM10_VLED+
- net /Terminal Blocks/DIMMER_OUT_5.4 renamed DIM10_VLED-
- net /Terminal Blocks/GND_VDC1 renamed GND_DIM1
- C1 pad 2: GND -> VIN_DIM1
- C10 pad 1: GND -> VIN_DIM1
- C11 pad 2: GND -> VIN_DIM1
- C12 pad 2: GND -> VIN_DIM1
- C13 pad 2: GND -> VIN_DIM1
- C15 pad 2: GND -> VIN_DIM1
- C16 pad 2: GND -> VIN_DIM1
- C17 pad 2: GND -> VIN_DIM1
- C18 pad 2: GND -> VIN_DIM1
- C19 pad 2: GND -> VIN_DIM1
- C2 pad 2: GND -> VIN_DIM1
- C20 pad 2: GND -> VIN_DIM1
- C21 pad 2: GND -> VIN_DIM1
- C3 pad 2: GND -> VIN_DIM1
- C4 pad 2: GND -> VIN_DIM1
- C5 pad 2: GND -> VIN_DIM1
- C6 pad 2: GND -> VIN_DIM1
- C7 pad 2: GND -> VIN_DIM1
- C8 pad 2: GND -> VIN_DIM1
- C9 pad 2: GND -> VIN_DIM1
- D1 pad 2: GND -> VIN_DIM1
- IC1 pad 17: GND -> VIN_DIM1
- IC1 pad 20: GND -> VIN_DIM1
- IC1 pad 22: GND -> VIN_DIM1
- IC1 pad 27: GND -> VIN_DIM1
- IC1 pad 29: GND -> VIN_DIM1
- IC1 pad 9: GND -> VIN_DIM1
- J1 pad 10: /Terminal Blocks/DIMMER_OUT_1.2 -> DIM1_VLED-
- J1 pad 11: /Terminal Blocks/DIMMER_OUT_1.3 -> DIM2_VLED+
- J1 pad 12: /Terminal Blocks/DIMMER_OUT_1.4 -> DIM2_VLED-
- J1 pad 2: GND -> VIN_DIM1
- J1 pad 7: /Terminal Blocks/VDC_IN1 -> VIN_DIM1
- J1 pad 9: /Terminal Blocks/DIMMER_OUT_1.1 -> DIM1_VLED+
- J2 pad 1: /Terminal Blocks/VDC_IN_2 -> VIN_DIM3
- J2 pad 2: /Terminal Blocks/GND_VDC_2 -> GND_DIM3
- J2 pad 7: /Terminal Blocks/VDC_IN_3 -> VIN_DIM5
- J2 pad 8: /Terminal Blocks/GND_VDC_3 -> GND_DIM5
- J3 pad 1: /Terminal Blocks/VDC_IN_4 -> VIN_DIM3
- J3 pad 2: /Terminal Blocks/GND_VDC_4 -> GND_DIM3
- J3 pad 7: /Terminal Blocks/VDC_IN_5 -> VIN_DIM5
- J3 pad 8: /Terminal Blocks/GND_VDC_5 -> GND_DIM5
- Q1 pad 2: GND -> VIN_DIM1
- Q2 pad 2: GND -> VIN_DIM1
- Q3 pad 2: GND -> VIN_DIM1
- Q4 pad 2: GND -> VIN_DIM1
- Q5 pad 2: GND -> VIN_DIM1
- Q6 pad 2: GND -> VIN_DIM1
- Q7 pad 2: GND -> VIN_DIM1
- Q9 pad 2: GND -> VIN_DIM1
- R12 pad 2: GND -> VIN_DIM1
- R15 pad 2: GND -> VIN_DIM1
- R16 pad 2: GND -> VIN_DIM1
- R17 pad 2: GND -> VIN_DIM1
- R2 pad 2: GND -> VIN_DIM1
- R21 pad 2: GND -> VIN_DIM1
- R4 pad 2: GND -> VIN_DIM1
- R9 pad 2: GND -> VIN_DIM1
Routing:
- added copper zone on F.Cu, net DIM1_VLED+
Other:
- board text added: "${REFERENCE}"

Commit message: layout for first dimmer
Parts:
- removed FRDM_MCXN947_1: MCU**, FRDM-MCXN947:FRDM-MCXN947
- added FRDM_MCXA153_1: MCU**, FFRDM-MCXA153:FRDM-MCXA153-SMD, F.Cu at (80.8, 68.7)
- C22, C29: footprint Capacitor_SMD:C_0201_0603Metric -> Capacitor_SMD:C_0603_1608Metric; moved to B.Cu
- C24, C25, C26, R38, R39, RS_DIM1, U1: moved to B.Cu
- C33, C35: footprint Capacitor_SMD:C_0201_0603Metric -> Capacitor_SMD:C_0603_1608Metric
- K1, K2, K3, K4, K5, K6, K7, K9: footprint Relays:20715562 -> Relay:20715562
- moved K7 127.5 mm to (-87.8, 109.3)
- moved K1 109.7 mm to (-111.1, 109.3), turned to 0 degrees
- moved K9 103.2 mm to (-87.8, 122.7)
- moved K2 89.0 mm to (-111.1, 122.7)
- moved K3 87.2 mm to (-111.1, 135.9), turned to 0 degrees
- moved K5 69.9 mm to (-111.1, 162.6), turned to 0 degrees
- moved D21 59.3 mm to (68.3, 103.1), turned to 180 degrees
- moved D20 58.7 mm to (74.2, 109.2), turned to -90 degrees
- moved K6 58.6 mm to (-111.1, 175.8), turned to 0 degrees
- moved K4 57.2 mm to (-111.1, 149.2)
- moved RS_DIM1 56.4 mm to (86.6, 113.2), turned to 90 degrees
- moved C22 54.9 mm to (71.1, 112.5), turned to -90 degrees
- moved C29 52.8 mm to (75.7, 117.6)
- moved U1 47.3 mm to (75.7, 113.0), turned to -90 degrees
- moved R39 38.8 mm to (79.8, 112.1), turned to 90 degrees
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Connections:
- net /Terminal Blocks/ANALOG_IN_1 renamed ANALOG_IN_1
- net /Terminal Blocks/ANALOG_IN_2 renamed ANALOG_IN_2
- net /Terminal Blocks/RS485_A renamed RS485_A
- net /Terminal Blocks/RS485_B renamed RS485_B
- net /Terminal Blocks/VDC_CTRL renamed VDC_CTRL
- net DIM10_VLED+ renamed DIM10_VLED_VCC
- net DIM10_VLED- renamed DIM10_VLED_GND
- net DIM1_VLED+ renamed DIM1_VLED_VCC
- net DIM1_VLED- renamed DIM1_VLED_GND
- net DIM2_VLED+ renamed DIM2_VLED_VCC
- net DIM2_VLED- renamed DIM2_VLED_GND
- net DIM3_VLED+ renamed DIM3_VLED_VCC
- net DIM3_VLED- renamed DIM3_VLED_GND
- net DIM4_VLED+ renamed DIM4_VLED_VCC
- net DIM4_VLED- renamed DIM4_VLED_GND
- net DIM5_VLED+ renamed DIM5_VLED_VCC
- net DIM5_VLED- renamed DIM5_VLED_GND
- net DIM6_VLED+ renamed DIM6_VLED_VCC
- net DIM6_VLED- renamed DIM6_VLED_GND
- net DIM7_VLED+ renamed DIM7_VLED_VCC
- net DIM7_VLED- renamed DIM7_VLED_GND
- net DIM8_VLED+ renamed DIM8_VLED_VCC
- net DIM8_VLED- renamed DIM8_VLED_GND
- net DIM9_VLED+ renamed DIM9_VLED_VCC
- net DIM9_VLED- renamed DIM9_VLED_GND
- net Net-(D20-A) renamed /Dimmer1/DIM1_FB
- net Net-(D21-K) renamed /Dimmer1/DIM1_SW
- net VAC_OUT_1.1 renamed VAC_OUT_1
- net VAC_OUT_9.1 renamed VAC_OUT_9
- C1 pad 2: VIN_DIM1 -> GND_CTRL
- C10 pad 1: VIN_DIM1 -> GND_CTRL
- C11 pad 2: VIN_DIM1 -> GND_CTRL
- C12 pad 2: VIN_DIM1 -> GND_CTRL
- C13 pad 2: VIN_DIM1 -> GND_CTRL
- C15 pad 2: VIN_DIM1 -> GND_CTRL
- C16 pad 2: VIN_DIM1 -> GND_CTRL
- C17 pad 2: VIN_DIM1 -> GND_CTRL
- C18 pad 2: VIN_DIM1 -> GND_CTRL
- C19 pad 2: VIN_DIM1 -> GND_CTRL
- C2 pad 2: VIN_DIM1 -> GND_CTRL
- C20 pad 2: VIN_DIM1 -> GND_CTRL
- C21 pad 2: VIN_DIM1 -> GND_CTRL
- C23 pad 2: VIN_DIM1 -> GND_CTRL
- C25 pad 2: VIN_DIM1 -> GND_CTRL
- C26 pad 2: VIN_DIM1 -> GND_CTRL
- C27 pad 2: VIN_DIM1 -> GND_CTRL
- C28 pad 2: VIN_DIM1 -> GND_CTRL
- C29 pad 2: VIN_DIM1 -> GND_CTRL
- C3 pad 2: VIN_DIM1 -> GND_CTRL
- C30 pad 2: VIN_DIM1 -> GND_CTRL
- C31 pad 2: VIN_DIM1 -> GND_CTRL
- C32 pad 2: VIN_DIM1 -> GND_CTRL
- C33 pad 2: VIN_DIM1 -> GND_CTRL
- C34 pad 2: VIN_DIM1 -> GND_CTRL
- C36 pad 2: VIN_DIM1 -> GND_CTRL
- C4 pad 2: VIN_DIM1 -> GND_CTRL
- C5 pad 2: VIN_DIM1 -> GND_CTRL
- C6 pad 2: VIN_DIM1 -> GND_CTRL
- C7 pad 2: VIN_DIM1 -> GND_CTRL
- C8 pad 2: VIN_DIM1 -> GND_CTRL
- C9 pad 2: VIN_DIM1 -> GND_CTRL
- D1 pad 2: VIN_DIM1 -> GND_CTRL
- D21 pad 2: VIN_DIM1 -> GND_CTRL
- D22 pad 2: VIN_DIM1 -> GND_CTRL
- IC1 pad 17: VIN_DIM1 -> GND_CTRL
- IC1 pad 20: VIN_DIM1 -> GND_CTRL
- IC1 pad 22: VIN_DIM1 -> GND_CTRL
- IC1 pad 27: VIN_DIM1 -> GND_CTRL
- IC1 pad 29: VIN_DIM1 -> GND_CTRL
- IC1 pad 9: VIN_DIM1 -> GND_CTRL
- J1 pad 2: VIN_DIM1 -> GND_CTRL
- J1 pad 8: GND_DIM1 -> GND_CTRL
- J4 pad 3: VAC_OUT_1.2 -> unconnected-(J4-Pin_3-Pad3)
- J4 pad 5: VAC_OUT_2.1 -> VAC_OUT_2
- J4 pad 6: VAC_OUT_2.2 -> unconnected-(J4-Pin_6-Pad6)
- J4 pad 8: VAC_OUT_3.1 -> VAC_OUT_3
- J4 pad 9: VAC_OUT_3.2 -> unconnected-(J4-Pin_9-Pad9)
- J5 pad 2: VAC_OUT_4.1 -> VAC_OUT_4
- J5 pad 3: VAC_OUT_4.2 -> unconnected-(J5-Pin_3-Pad3)
- J5 pad 5: VAC_OUT_5.1 -> VAC_OUT_5
- J5 pad 6: VAC_OUT_5.2 -> unconnected-(J5-Pin_6-Pad6)
- J5 pad 8: VAC_OUT_6.1 -> VAC_OUT_6
- J5 pad 9: VAC_OUT_6.2 -> unconnected-(J5-Pin_9-Pad9)
- J6 pad 2: VAC_OUT_7.1 -> VAC_OUT_7
- J6 pad 3: VAC_OUT_7.2 -> unconnected-(J6-Pin_3-Pad3)
- J6 pad 5: VAC_OUT_8.1 -> VAC_OUT_8
- J6 pad 6: VAC_OUT_8.2 -> unconnected-(J6-Pin_6-Pad6)
- J6 pad 9: VAC_OUT_9.2 -> unconnected-(J6-Pin_9-Pad9)
- K2 pad 3: VAC_OUT_1.2 -> VAC_OUT_2
- K2 pad 4: VAC_IN_1 -> VAC_IN_2
- K3 pad 3: VAC_OUT_2.1 -> VAC_OUT_3
- K3 pad 4: VAC_IN_2 -> VAC_IN_3
- K4 pad 3: VAC_OUT_2.2 -> VAC_OUT_4
- K4 pad 4: VAC_IN_2 -> VAC_IN_4
- K5 pad 3: VAC_OUT_3.1 -> VAC_OUT_5
- K5 pad 4: VAC_IN_3 -> VAC_IN_5
- K6 pad 3: VAC_OUT_3.2 -> VAC_OUT_6
- K6 pad 4: VAC_IN_3 -> VAC_IN_6
- K7 pad 3: VAC_OUT_4.1 -> VAC_OUT_7
- K7 pad 4: VAC_IN_4 -> VAC_IN_7
- K9 pad 3: VAC_OUT_5.1 -> VAC_OUT_8
- K9 pad 4: VAC_IN_5 -> VAC_IN_8
- Q1 pad 2: VIN_DIM1 -> GND_CTRL
- Q2 pad 2: VIN_DIM1 -> GND_CTRL
- Q3 pad 2: VIN_DIM1 -> GND_CTRL
- Q4 pad 2: VIN_DIM1 -> GND_CTRL
- Q5 pad 2: VIN_DIM1 -> GND_CTRL
- Q6 pad 2: VIN_DIM1 -> GND_CTRL
- Q7 pad 2: VIN_DIM1 -> GND_CTRL
- Q9 pad 2: VIN_DIM1 -> GND_CTRL
- R12 pad 2: VIN_DIM1 -> GND_CTRL
- R15 pad 2: VIN_DIM1 -> GND_CTRL
- R16 pad 2: VIN_DIM1 -> GND_CTRL
- R17 pad 2: VIN_DIM1 -> GND_CTRL
- R2 pad 2: VIN_DIM1 -> GND_CTRL
- R21 pad 2: VIN_DIM1 -> GND_CTRL
- R4 pad 2: VIN_DIM1 -> GND_CTRL
- R9 pad 2: VIN_DIM1 -> GND_CTRL
- RS_DIM1 pad 2: VIN_DIM1 -> GND_CTRL
- RS_DIM2 pad 2: VIN_DIM1 -> GND_CTRL
- U1 pad 6: VIN_DIM1 -> GND_CTRL
- U1 pad 9: VIN_DIM1 -> GND_CTRL
- U2 pad 6: VIN_DIM1 -> GND_CTRL
- U2 pad 9: VIN_DIM1 -> GND_CTRL
Routing:
- net /Dimmer1/DIM1_SW: track 0.00 -> 34.6 mm, vias 0 -> 6
- net DIM1_VLED_GND: track 0.00 -> 28.7 mm, vias 0 -> 1
- net GND_CTRL: track 0.00 -> 27.8 mm, vias 0 -> 12
- net DIM1_VLED_VCC: track 0.00 -> 26.6 mm, vias 0 -> 8
- net /Dimmer1/DIM1_FB: track 0.00 -> 11.4 mm, vias 0 -> 1
- net VIN_DIM1: track 0.00 -> 9.20 mm
- net PWM_DIM1: track 0.00 -> 4.68 mm, vias 0 -> 1
- net Net-(U1-COMP): track 0.00 -> 3.79 mm
- net Net-(U1-BOOT): track 0.00 -> 3.25 mm
- net Net-(C26-Pad1): track 0.00 -> 1.83 mm
- net INH_DIM1: track 0.00 -> 1.71 mm, vias 0 -> 1
- added copper zone on B.Cu, net /Dimmer1/DIM1_SW
- added copper zone on F.Cu, net /Dimmer1/DIM1_SW
- added copper zone on B.Cu, net DIM1_VLED_VCC
- added copper zone on B.Cu, net VIN_DIM1
