File: io-gateway/io-gateway.kicad_pcb (KiCad board)
At the start: 4 copper layers, 155 x 81.5 mm, 120 parts, among them J1 1752201, J2 1752201, J3 1752201, J4 Screw_Terminal_01x09, J5 Screw_Terminal_01x09, J6 Screw_Terminal_01x09, K1 2071556-2, K2 2071556-2, K3 2071556-2, K4 2071556-2, K5 2071556-2, K6 2071556-2, K7 2071556-2, K8 2071556-2, K9 2071556-2, U3 TPS54308

Commit message: duplicate dimmer
Parts:
- C_DIMA_11, C_DIMA_12, C_DIMA_13, C_DIMA_14, C_DIMA_15, C_DIMA_16, C_DIMB_10, C_DIMB_11, C_DIMB_12, C_DIMB_13, C_DIMB_14, C_DIMB_15, C_DIMB_9, D_DIMB_4, RS_DIMA_2, RS_DIMB_2, R_DIMA_3, R_DIMA_4, R_DIMB_3, R_DIMB_4, U_DIMA2, U_DIMB2: moved to B.Cu
- moved D_DIMB_3 232.5 mm to (105.2, 63.2), turned to -90 degrees
- moved D_DIMA_3 231.8 mm to (67.7, 71.0), turned to 180 degrees
- moved D_DIMA_4 227.5 mm to (73.5, 77.1), turned to -90 degrees
- moved D_DIMB_4 227.1 mm to (105.1, 72.7), turned to -90 degrees
- moved L_DIMB_2 223.2 mm to (92.5, 66.4), turned to 90 degrees
- moved RS_DIMB_2 222.8 mm to (93.1, 81.1), turned to 90 degrees
- moved C_DIMA_14 222.3 mm to (70.5, 80.4), turned to -90 degrees
- moved RS_DIMA_2 220.3 mm to (84.9, 82.8)
- moved R_DIMB_3 220.1 mm to (100.7, 73.5), turned to -90 degrees
- moved C_DIMA_13 220.1 mm to (79.1, 77.3)
- moved C_DIMB_13 219.7 mm to (98.5, 73.5), turned to 90 degrees
- moved C_DIMB_14 215.5 mm to (95.2, 81.1), turned to -90 degrees
- moved R_DIMA_3 215.5 mm to (79.1, 79.9), turned to 90 degrees
- moved C_DIMB_11 213.8 mm to (102.7, 73.5), turned to -90 degrees
- moved R_DIMA_4 213.5 mm to (79.4, 84.5), turned to 90 degrees
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Connections:
- C_DIMA_15 pad 1: /Dimmer2/DIM_VLED+_A -> DIM3_VLED_VCC
- C_DIMA_16 pad 1: /Dimmer2/DIM_VLED+_A -> DIM3_VLED_VCC
- C_DIMA_16 pad 2: /Dimmer2/DIM_VLED-_A -> DIM3_VLED_GND
- C_DIMB_15 pad 1: /Dimmer2/DIM_VLED+_B -> DIM4_VLED_VCC
- C_DIMB_16 pad 1: /Dimmer2/DIM_VLED+_B -> DIM4_VLED_VCC
- C_DIMB_16 pad 2: /Dimmer2/DIM_VLED-_B -> DIM4_VLED_GND
- D_DIMA_4 pad 1: /Dimmer2/DIM_VLED+_A -> DIM3_VLED_VCC
- D_DIMB_4 pad 1: /Dimmer2/DIM_VLED+_B -> DIM4_VLED_VCC
- J2 pad 1: VIN_DIM3 -> /Dimmer2/VIN_DIM
- J2 pad 2: GND_DIM3 -> GND_CTRL
- L_DIMA_2 pad 1: /Dimmer2/DIM_VLED+_A -> DIM3_VLED_VCC
- L_DIMB_2 pad 1: /Dimmer2/DIM_VLED+_B -> DIM4_VLED_VCC
- RS_DIMA_2 pad 1: /Dimmer2/DIM_VLED-_A -> DIM3_VLED_GND
- RS_DIMB_2 pad 1: /Dimmer2/DIM_VLED-_B -> DIM4_VLED_GND
- R_DIMA_4 pad 1: /Dimmer2/DIM_VLED-_A -> DIM3_VLED_GND
- R_DIMB_4 pad 1: /Dimmer2/DIM_VLED-_B -> DIM4_VLED_GND
Routing:
- net +5V: track 133.3 -> 20.2 mm
- net /Dimmer2/VIN_DIM: track 0.00 -> 88.8 mm, vias 0 -> 7
- net DIM4_VLED_GND: track 0.00 -> 87.4 mm, vias 0 -> 4
- net DIM4_VLED_VCC: track 0.00 -> 84.0 mm, vias 0 -> 12
- net DIM3_VLED_VCC: track 0.00 -> 82.4 mm, vias 0 -> 8
- net DIM3_VLED_GND: track 0.00 -> 75.4 mm, vias 0 -> 3
- net GND_CTRL: track 64.4 -> 121.6 mm, vias 28 -> 49
- net /Dimmer2/DIM2_SW: track 0.00 -> 48.8 mm, vias 0 -> 14
- net /Dimmer2/DIM1_SW: track 0.00 -> 34.6 mm, vias 0 -> 6
- net /Dimmer2/DIM1_FB: track 0.00 -> 14.3 mm, vias 0 -> 1
- net /Dimmer2/DIM2_FB: track 0.00 -> 12.6 mm
- net /Dimmer2/INH_DIMB: track 0.00 -> 6.69 mm, vias 0 -> 1
- net Net-(U_DIMB2-COMP): track 0.00 -> 6.46 mm
- net /Dimmer1/DIM2_SW: track 37.2 -> 42.7 mm
- net Net-(U_DIMB2-BOOT): track 0.00 -> 5.10 mm
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- added copper zone on B.Cu, net /Dimmer2/DIM1_SW
- added copper zone on F.Cu, net /Dimmer2/DIM1_SW
- added copper zone on B.Cu, net /Dimmer2/DIM2_SW
- added copper zone on F.Cu, net /Dimmer2/DIM2_SW
- added copper zone on In2.Cu, net /Dimmer2/DIM2_SW
- added copper zone on B.Cu, net /Dimmer2/VIN_DIM
- added copper zone on In2.Cu, net DIM3_VLED_GND
- added copper zone on B.Cu, net DIM3_VLED_VCC
- added copper zone on F.Cu, net DIM3_VLED_VCC
- added copper zone on B.Cu, net DIM4_VLED_GND
- added copper zone on In2.Cu, net DIM4_VLED_GND
- added copper zone on B.Cu, net DIM4_VLED_VCC
- added copper zone on F.Cu, net DIM4_VLED_VCC
- added copper zone on In2.Cu, net DIM4_VLED_VCC

Commit message: Place some Relays
Parts:
- removed C44: 47µF, Capacitor_SMD:CP_Elec_6.3x5.4
- D_DIMA_3, D_K1, D_K2, D_K3, Q_K1, Q_K2, Q_K3, R_K1, R_K2, R_K3: moved to B.Cu
- F1: footprint Fuse:Fuseholder_Cylinder-5x20mm_Wuerth_696103101002-SMD_Horizontal_Open -> Fuse:Fuse_0603_1608Metric
- moved K6 236.8 mm to (118.0, 92.8), turned to 180 degrees
- moved K2 214.1 mm to (68.8, 74.6), turned to 180 degrees
- moved D_K2 213.3 mm to (67.8, 78.7), turned to -90 degrees
- moved K4 211.5 mm to (122.8, 147.1), turned to 180 degrees
- moved D_K3 210.5 mm to (68.8, 65.7), turned to -90 degrees
- moved K3 210.4 mm to (68.8, 61.7), turned to 180 degrees
- moved Q_K2 205.1 mm to (64.1, 80.4)
- moved Q_K3 200.9 mm to (64.8, 69.3)
- moved R_K2 197.6 mm to (60.5, 80.5), turned to -90 degrees
- moved R_K3 193.2 mm to (61.1, 69.5), turned to -90 degrees
- moved K1 181.3 mm to (68.8, 87.4), turned to 180 degrees
- moved D_K1 178.0 mm to (68.8, 91.3), turned to -90 degrees
- moved Q_K1 174.6 mm to (64.9, 95.0)
- moved R_K1 166.0 mm to (61.0, 95.1), turned to -90 degrees
- moved C41 35.8 mm to (58.9, 99.1), turned to 90 degrees
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Routing:
- net /Dimmer2/DIM1_SW: track 34.6 -> 46.3 mm, vias 6 -> 5
- net Net-(D_K3-A): track 0.00 -> 4.95 mm
- net Net-(D_K1-A): track 0.00 -> 4.83 mm
- net Net-(D_K2-A): track 0.00 -> 4.80 mm
- net DIM3_VLED_GND: track 75.4 -> 79.8 mm
- net VDC_CTRL: track 12.4 -> 8.90 mm
- net +24V: track 16.2 -> 19.5 mm
- net Net-(Q_K1-G): track 0.00 -> 2.81 mm
- net /MCU_VoltageRegulator/VregSW: track 15.0 -> 17.7 mm
- net DIM4_VLED_GND: track 87.4 -> 89.9 mm, vias 4 -> 5
- net Net-(Q_K2-G): track 0.00 -> 2.55 mm
- net Net-(Q_K3-G): track 0.00 -> 2.55 mm
- net +5V: track 20.2 -> 18.3 mm
- net /Relay2/SW_IN: track 0.00 -> 1.59 mm, vias 0 -> 1
- net /Dimmer1/DIM1_SW: track 34.6 -> 33.1 mm
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
Commit message: fix some drc issues
Parts:
- added C44: 47µF, Capacitor_SMD:CP_Elec_6.3x5.4, F.Cu at (55.5, 104.0)
- added C_DIMA_17: 10µF 50V, Capacitor_SMD:C_1210_3225Metric, F.Cu at (129.0, 114.0)
- added C_DIMA_18: 10µF 50V, Capacitor_SMD:C_1210_3225Metric, F.Cu at (125.4, 114.0)
- added C_DIMA_19: 470pF, Capacitor_SMD:C_0603_1608Metric, B.Cu at (134.8, 113.5)
- added C_DIMA_20: 100nF 50V, Capacitor_SMD:C_0603_1608Metric, B.Cu at (129.0, 117.6)
- added C_DIMA_21: 22pF, Capacitor_SMD:C_0603_1608Metric, B.Cu at (133.0, 109.5)
- added C_DIMA_22: 100nF 50V, Capacitor_SMD:C_0603_1608Metric, B.Cu at (124.4, 112.5)
- added C_DIMA_23: 1µF 50V, Capacitor_SMD:C_1206_3216Metric, B.Cu at (129.4, 103.4)
- added C_DIMA_24: NM, Capacitor_SMD:C_1206_3216Metric, B.Cu at (138.3, 117.1)
- added C_DIMB_17: 10µF 50V, Capacitor_SMD:C_1210_3225Metric, B.Cu at (161.3, 116.3)
- added C_DIMB_18: 10µF 50V, Capacitor_SMD:C_1210_3225Metric, B.Cu at (161.3, 112.8)
- added C_DIMB_19: 470pF, Capacitor_SMD:C_0603_1608Metric, B.Cu at (156.6, 105.6)
- added C_DIMB_20: 100nF 50V, Capacitor_SMD:C_0603_1608Metric, B.Cu at (155.3, 118.8)
- added C_DIMB_21: 22pF, Capacitor_SMD:C_0603_1608Metric, B.Cu at (152.4, 105.6)
- added C_DIMB_22: 100nF 50V, Capacitor_SMD:C_0603_1608Metric, B.Cu at (149.1, 113.2)
- added C_DIMB_23: 1µF 50V, Capacitor_SMD:C_1206_3216Metric, B.Cu at (140.4, 106.1)
- added C_DIMB_24: NM, Capacitor_SMD:C_1206_3216Metric, F.Cu at (151.3, 125.6)
- added D_DIMA_5: D_Schottky, Diode_SMD:D_SMB, F.Cu at (115.7, 109.2)
- added D_DIMA_6: D_Zener, Diode_SMD:D_SOD-123, F.Cu at (127.4, 109.2)
- added D_DIMB_5: D_Schottky, Diode_SMD:D_SMB, F.Cu at (156.3, 97.3)
- added D_DIMB_6: D_Zener, Diode_SMD:D_SOD-123, B.Cu at (159.0, 104.8)
- added L_DIMA_3: 47µH 3.8A, Inductor_SMD:L_12x12mm_H8mm, F.Cu at (133.0, 98.5)
- added L_DIMB_3: 47µH 3.8A, Inductor_SMD:L_12x12mm_H8mm, F.Cu at (146.4, 98.4)
- added RS_DIMA_3: R, Resistor_SMD:R_1206_3216Metric, B.Cu at (139.9, 113.2)
- added RS_DIMB_3: R, Resistor_SMD:R_1206_3216Metric, B.Cu at (147.0, 113.2)
- added R_DIMA_5: 24k9, Resistor_SMD:R_0603_1608Metric, B.Cu at (133.0, 112.1)
- added R_DIMA_6: 47k, Resistor_SMD:R_0603_1608Metric, B.Cu at (133.3, 116.6)
- added R_DIMB_5: 24k9, Resistor_SMD:R_0603_1608Metric, B.Cu at (154.6, 105.6)
- added R_DIMB_6: 47k, Resistor_SMD:R_0603_1608Metric, B.Cu at (157.4, 115.7)
- added U_DIMA3: LED5000, Package_SO:HSOP-8-1EP_3.9x4.9mm_P1.27mm_EP2.41x3.1mm, B.Cu at (129.0, 113.0)
- added U_DIMB3: LED5000, Package_SO:HSOP-8-1EP_3.9x4.9mm_P1.27mm_EP2.41x3.1mm, B.Cu at (152.9, 113.3)
- C_DIMA_10, C_DIMA_9: moved to B.Cu
- moved K5 127.5 mm to (26.6, 114.8)
- moved K4 94.1 mm to (28.9, 141.2)
- moved C_DIMA_10 11.9 mm to (78.2, 91.7), turned to -90 degrees
- moved C_DIMA_9 10.0 mm to (73.4, 91.8), turned to -90 degrees
Connections:
- FRDM_MCXA153_1 pad 3.12: unconnected-(FRDM_MCXA153_1B-Pin_J3_12_GND-Pad3.12) -> GND_CTRL
- FRDM_MCXA153_1 pad 3.14: unconnected-(FRDM_MCXA153_1B-Pin_J3_14_GND-Pad3.14) -> GND_CTRL
- FRDM_MCXA153_1 pad 3.16: unconnected-(FRDM_MCXA153_1B-Pin_J3_16_VIN-Pad3.16) -> +5V
- J2 pad 7: VIN_DIM5 -> /Dimmer3/VIN_DIM
- J2 pad 8: GND_DIM5 -> GND_CTRL
Routing:
- net GND_CTRL: track 121.6 -> 198.7 mm, vias 49 -> 68
- net DIM6_VLED_VCC: track 0.00 -> 50.3 mm, vias 0 -> 4
- net /Dimmer3/VIN_DIM: track 0.00 -> 49.1 mm, vias 0 -> 12
- net /Dimmer3/DIM1_SW: track 0.00 -> 34.6 mm, vias 0 -> 6
- net DIM5_VLED_VCC: track 0.00 -> 33.4 mm, vias 0 -> 8
- net DIM6_VLED_GND: track 0.00 -> 32.5 mm, vias 0 -> 1
- net /Dimmer3/DIM2_SW: track 0.00 -> 30.6 mm, vias 0 -> 11
- net DIM5_VLED_GND: track 0.00 -> 23.4 mm, vias 0 -> 1
- net /Dimmer3/DIM1_FB: track 0.00 -> 14.3 mm, vias 0 -> 1
- net /Dimmer3/DIM2_FB: track 0.00 -> 12.1 mm
- net /Dimmer2/DIM2_SW: track 48.8 -> 40.0 mm
- net /Dimmer2/VIN_DIM: track 88.8 -> 96.5 mm
- net /Dimmer3/INH_DIMB: track 0.00 -> 6.98 mm, vias 0 -> 1
- net Net-(U_DIMB3-COMP): track 0.00 -> 6.46 mm
- net Net-(U_DIMB3-BOOT): track 0.00 -> 6.18 mm
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- added copper zone on B.Cu, net (none)
- added copper zone on F.Cu, net +5V
- added copper zone on B.Cu, net /Dimmer1/DIM1_FB
- added copper zone on B.Cu, net /Dimmer3/DIM1_FB
- added copper zone on B.Cu, net /Dimmer3/DIM1_SW
- added copper zone on F.Cu, net /Dimmer3/DIM1_SW
- added copper zone on B.Cu, net /Dimmer3/DIM2_SW
- added copper zone on F.Cu, net /Dimmer3/DIM2_SW
- added copper zone on In2.Cu, net /Dimmer3/DIM2_SW
- added copper zone on B.Cu, net /Dimmer3/VIN_DIM
- added copper zone on In2.Cu, net /Dimmer3/VIN_DIM
- added copper zone on B.Cu, net DIM5_VLED_VCC
- added copper zone on F.Cu, net DIM5_VLED_VCC
- added copper zone on B.Cu, net DIM6_VLED_VCC
- added copper zone on F.Cu, net DIM6_VLED_VCC
- added copper zone on In1.Cu, net GND_CTRL
- removed copper zone on F.Cu, net unconnected-(FRDM_MCXA153_1B-Pin_J3_16_VIN-Pad3.16)
Other:
- board text removed: "${REFERENCE}"

Commit message: Connect some Relays
Parts:
- moved R_K3 15.3 mm to (76.2, 67.2), turned to 90 degrees
- moved R_K1 12.6 mm to (73.0, 98.8)
- moved Q_K3 8.00 mm to (72.5, 67.3), turned to 180 degrees
- moved Q_K1 5.30 mm to (68.8, 98.5), turned to 90 degrees
- moved L6 1.83 mm to (63.1, 105.2)
Routing:
- net /VAC_OUT_1.1: track 0.00 -> 76.8 mm
- net /VAC_IN_1: track 0.00 -> 75.4 mm
- net /Relay6/VAC_IN: track 0.00 -> 56.6 mm
- net /VAC_IN_2: track 0.00 -> 51.1 mm
- net /Relay6/VAC_OUT: track 0.00 -> 46.7 mm, vias 0 -> 1
- net /VAC_OUT_2.1: track 0.00 -> 33.3 mm
- net /Dimmer2/DIM1_SW: track 45.5 -> 16.6 mm
- net /VAC_IN_3: track 0.00 -> 23.0 mm
- net /VAC_OUT_3.1: track 0.00 -> 11.5 mm
- net /MCU_VoltageRegulator/VregFB: track 11.5 -> 6.32 mm
- net Net-(U3-EN): track 19.7 -> 15.3 mm
- net DIM4_VLED_VCC: track 84.0 -> 86.5 mm, vias 12 -> 10
- net /MCU_VoltageRegulator/VregSW: track 17.7 -> 15.2 mm
- net GND_CTRL: track 198.7 -> 196.7 mm, vias 68 -> 67
- net /Dimmer2/VIN_DIM: track 96.5 -> 98.0 mm
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