File: io-gateway/dimmer1.kicad_sch (KiCad schematic)
At the start: 34 parts

Commit message: upd
Parts:
- D_DIMA_2: footprint Diode_SMD:D_SOD-123 -> D_SOD-123:D_SOD-123
- RS_DIMA_2: footprint Resistor_SMD:R_1206_3216Metric -> Resistor_SMD:R_1206_3216Metric_Pad1.30x1.75mm_HandSolder
Changed lines of the file:
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@@
 			)
 		)
-		(property "Footprint" "Resistor_SMD:R_1206_3216Metric"
+		(property "Footprint" "Resistor_SMD:R_1206_3216Metric_Pad1.30x1.75mm_HandSolder"
 			(at 197.358 72.39 90)
 			(effects
@@
 			)
 		)
-		(property "Footprint" "Diode_SMD:D_SOD-123"
+		(property "Footprint" "D_SOD-123:D_SOD-123"
 			(at 158.75 54.61 0)
 			(effects

Commit message: add fuses to Dimmer VIN
Parts:
- added F_DIMA_1: Fuse, Fuse:Fuse_1206_3216Metric_Pad1.42x1.75mm_HandSolder, symbol Device:Fuse
Connections:
- net VIN_DIM: now also F_DIMA_1.1; no longer C_DIMA_1.1, C_DIMA_2.1, C_DIMA_3.1, U_DIMA1.7 (VIN)
- new net: C_DIMA_1.1, C_DIMA_2.1, C_DIMA_3.1, F_DIMA_1.2, U_DIMA1.7 (VIN)
Changed lines of the file:
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@@
 	)
 	(junction
-		(at 43.18 21.59)
+		(at 132.08 80.01)
 		(diameter 0)
 		(color 0 0 0 0)
 	)
 	(junction
-		(at 132.08 80.01)
+		(at 82.55 154.94)
 		(diameter 0)
 		(color 0 0 0 0)
 	)
 	(junction
-		(at 82.55 154.94)
+		(at 43.18 35.56)
 		(diameter 0)
 		(color 0 0 0 0)
 	)
 	(junction
-		(at 43.18 35.56)
+		(at 43.18 21.59)
 		(diameter 0)
 		(color 0 0 0 0)
@@
 	(wire
 		(pts
+			(xy 26.67 21.59) (xy 21.59 21.59)
+		)
+		(stroke
+			(width 0)
+			(type default)
+		)
+	)
+	(wire
+		(pts
 			(xy 176.53 154.94) (xy 194.31 154.94)
 		)
@@
 	(wire
 		(pts
-			(xy 43.18 21.59) (xy 43.18 25.4)
+			(xy 34.29 21.59) (xy 43.18 21.59)
 		)
 		(stroke
@@
 	(wire
 		(pts
-			(xy 21.59 21.59) (xy 43.18 21.59)
-		)
-		(stroke
-			(width 0)
-			(type default)
-		)
-	)
-	(wire
-		(pts
 			(xy 201.93 46.99) (xy 205.74 46.99)
 		)
@@
 	(wire
 		(pts
+			(xy 43.18 21.59) (xy 43.18 25.4)
+		)
+		(stroke
+			(width 0)
+			(type default)
+		)
+	)
+	(wire
+		(pts
 			(xy 24.13 46.99) (xy 87.63 46.99)
 		)
@@
 					(unit 1)
 				)
+			)
+		)
+	)
+	(symbol
+		(lib_id "Device:Fuse")
+		(at 30.48 21.59 90)
+		(unit 1)
+		(exclude_from_sim no)
+		(in_bom yes)
+		(on_board yes)
+		(dnp no)
+		(fields_autoplaced yes)
+		(property "Reference" "F_DIMA_1"
+			(at 30.48 15.24 90)
+			(effects
+				(font
+					(size 1.27 1.27)
+				)
+			)
+		)
+		(property "Value" "Fuse"
+			(at 30.48 17.78 90)
+			(effects
+				(font
+					(size 1.27 1.27)
+				)
+			)
+		)
+		(property "Footprint" "Fuse:Fuse_1206_3216Metric_Pad1.42x1.75mm_HandSolder"
+			(at 30.48 23.368 90)
+			(effects
+				(font
+					(size 1.27 1.27)
+				)
+				(hide yes)
+			)
+		)
+		(property "Datasheet" "~"
+			(at 30.48 21.59 0)
+			(effects
+				(font
+					(size 1.27 1.27)
+				)
+				(hide yes)
+			)
+		)
+		(property "Description" "Fuse"
+			(at 30.48 21.59 0)
+			(effects
+				(font
+					(size 1.27 1.27)
+				)
+				(hide yes)
+			)
+		)
+		(pin "2"
+		)
+		(pin "1"
+		)
+		(instances
+			(project "io-gateway"
+				(path "/2cb6f94b-272a-4ed7-b08d-c3630bda6156/334a84ed-29ea-43c8-926f-91a0c21c840d"
+					(reference "F_DIMA_1")
+					(unit 1)
+				)
+				(path "/2cb6f94b-272a-4ed7-b08d-c3630bda6156/6816aaeb-2895-4813-8cf8-10286e1728b3"
+					(reference "F_DIMA_3")
+					(unit 1)
+				)
+				(path "/2cb6f94b-272a-4ed7-b08d-c3630bda6156/af08ab74-4e14-4265-a7c4-2b601284ca87"
+					(reference "F_DIMA_5")
+					(unit 1)
+				)
+				(path "/2cb6f94b-272a-4ed7-b08d-c3630bda6156/c5ad205a-3c42-42cf-b4c7-d7c0b439897b"
+					(reference "F_DIMA_4")
+					(unit 1)
+				)

Commit message: upd
Connections:
- net VIN_DIM: no longer C_DIMB_1.1, C_DIMB_2.1, C_DIMB_3.1, U_DIMB1.7 (VIN)
- net VIN_DIM_F: now reaches C_DIMA_1.1, C_DIMA_2.1, C_DIMA_3.1, F_DIMA_1.2, U_DIMA1.7 (VIN)
- net VIN_DIM_F: now also C_DIMB_1.1, C_DIMB_2.1, C_DIMB_3.1, U_DIMB1.7 (VIN)
Changed lines of the file:
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@@
 		)
 	)
-	(label "VIN_DIM"
+	(label "VIN_DIM_F"
 		(at 30.48 96.52 0)
 		(effects
@@
 		(effects
 			(font
+				(size 1.27 1.27)
+			)
+			(justify left bottom)
+		)
+	)
+	(label "VIN_DIM_F"
+		(at 38.1 21.59 0)
+		(effects
+			(font

Commit message: V1.2
Parts:
- C_DIMA_8, C_DIMB_8: value NM -> DNP
Changed lines of the file:
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@@
 			)
 		)
-		(property "Value" "NM"
+		(property "Value" "DNP"
 			(at 210.82 129.5399 0)
 			(effects
@@
 			)
 		)
-		(property "Value" "NM"
+		(property "Value" "DNP"
 			(at 209.55 54.6099 0)
 			(effects
